File: kicad/STM_Morpho/STM_Morpho.sch (KiCad schematic (older format))
At the start: 5 parts, among them CN10 CONN_02X19, CN7 CONN_02X19, J1 Conn_GameBoy_Cartridge_Slot, SW1 SW_SPDT, SW2 SW_SPST

Commit message: Use different GBA cart slot
Parts:
- CN10, CN7: symbol CONN_02X19 -> STM_Morpho-rescue:CONN_02X19
- J1: symbol Conn_GameBoy_Cartridge_Slot -> STM_Morpho-rescue:Conn_GameBoy_Cartridge_Slot
- SW1: symbol SW_SPDT -> STM_Morpho-rescue:SW_SPDT
- SW2: symbol SW_SPST -> STM_Morpho-rescue:SW_SPST
Changed lines of the file:
@@
-EESchema Schematic File Version 2
-LIBS:power
-LIBS:device
-LIBS:transistors
-LIBS:conn
-LIBS:linear
-LIBS:regul
-LIBS:74xx
-LIBS:cmos4000
-LIBS:adc-dac
-LIBS:memory
-LIBS:xilinx
-LIBS:microcontrollers
-LIBS:dsp
-LIBS:microchip
-LIBS:analog_switches
-LIBS:motorola
-LIBS:texas
-LIBS:intel
-LIBS:audio
-LIBS:interface
-LIBS:digital-audio
-LIBS:philips
-LIBS:display
-LIBS:cypress
-LIBS:siliconi
-LIBS:opto
-LIBS:atmel
-LIBS:contrib
-LIBS:valves
-LIBS:Gekkio_GameBoy
-LIBS:switches
+EESchema Schematic File Version 4
 LIBS:STM_Morpho-cache
-EELAYER 25 0
+EELAYER 26 0
 EELAYER END
 $Descr A4 11693 8268
@@
 $EndDescr
 $Comp
-L CONN_02X19 CN7
+L STM_Morpho-rescue:CONN_02X19 CN7
 U 1 1 58745202
 P 3550 3050
@@
 $EndComp
 $Comp
-L CONN_02X19 CN10
+L STM_Morpho-rescue:CONN_02X19 CN10
 U 1 1 5874523E
 P 6750 3050
@@
 $EndComp
 $Comp
-L Conn_GameBoy_Cartridge_Slot J1
+L STM_Morpho-rescue:Conn_GameBoy_Cartridge_Slot J1
 U 1 1 5AAC96CF
 P 9650 3050
@@
 $EndComp
 $Comp
-L SW_SPDT SW1
+L STM_Morpho-rescue:SW_SPDT SW1
 U 1 1 5AAC9860
 P 7500 4600
@@
 $EndComp
 $Comp
-L SW_SPST SW2
+L STM_Morpho-rescue:SW_SPST SW2
 U 1 1 5AAC98D7
 P 7500 5400
@@
 NoConn ~ 7000 3950
 $Comp
-L GND #PWR01
+L STM_Morpho-rescue:GND #PWR01
 U 1 1 5AACE29A
 P 5950 5550
